File: Schematics/fameboy_button_pads.brd (EAGLE design)
At the start: 40 x 59 mm, 13 parts

Commit message: gerbers
Parts:
- S1: value SWITCH-MOMENTARY-2SIDE_EZ -> SWITCH-MOMENTARY-2SIDE; device SparkFun-Electromechanical:TACTILE-PTH-SIDEEZ -> SparkFun-Electromechanical:TACTILE-PTH-SIDE
Other:
- board text added: "11mm button spacing"
- board text added: "13mm apart"
- board text added: "16mm apart"
- board text added: "25 degrees"
- board text added: "25mm from center to center"
- board text added: "6mm"
Changed lines of the file:
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@@
 <text x="5.08" y="50.8" size="1.27" layer="25">MUCH BOARD</text>
 <text x="27.94" y="5.08" size="1.27" layer="25">SUCH WOW</text>
+<text x="30.988" y="16.764" size="1.27" layer="25" rot="R225">13mm apart</text>
+<text x="25.4" y="20.32" size="1.27" layer="26" rot="MR25">16mm apart</text>
+<text x="19.812" y="6.858" size="1.27" layer="26" rot="MR25">25 degrees</text>
+<text x="20.32" y="15.24" size="1.27" layer="26" rot="MR90">25mm from center to center</text>
+<text x="8.382" y="39.37" size="1.27" layer="25">11mm button spacing</text>
+<text x="25.908" y="46.228" size="1.27" layer="25" rot="R115">6mm</text>
+<text x="29.972" y="43.942" size="1.27" layer="25" rot="R205">6mm</text>
+<text x="12.7" y="48.514" size="1.27" layer="25" rot="R205">6mm</text>
 </plain>
 <attributes>
@@
 <element name="U$3" library="parts" package="SELECTSTART" value="SELECTSTART" x="20" y="45"/>
 <element name="U$4" library="parts" package="SELECTSTART" value="SELECTSTART" x="20" y="45" rot="MR0"/>
-<element name="S1" library="SparkFun-Electromechanical" package="TACTILE-PTH-SIDEEZ" value="SWITCH-MOMENTARY-2SIDE_EZ" x="34" y="57" rot="R180"/>
+<element name="S1" library="SparkFun-Electromechanical" package="TACTILE-PTH-SIDE" value="SWITCH-MOMENTARY-2SIDE" x="34" y="57" rot="R180"/>
 <element name="JP1" library="SparkFun-Connectors" package="1X08_ROUND" value="" x="11.1125" y="2.5"/>
 <element name="U$5" library="LOGOS" package="DAVEDARKO2_LOGO" value="" x="35.56" y="12.7" rot="MR0"/>

Commit message: double shoulder button
Parts:
- added S2: SWITCH-MOMENTARY-2SIDE, SparkFun-Electromechanical:TACTILE-PTH-SIDE
Connections:
- net C3: now also S2.1
- net R3: now also S2.2
Routing:
- net C3: track 113.7 -> 142.9 mm
- net R3: track 169.1 -> 178.7 mm
Changed lines of the file:
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@@
 <setting verticaltext="up"/>
 </settings>
-<grid distance="0.1" unitdist="inch" unit="inch" style="lines" multiple="1" display="yes" altdistance="0.01" altunitdist="inch" altunit="inch"/>
+<grid distance="1" unitdist="mm" unit="mm" style="lines" multiple="1" display="yes" altdistance="0.1" altunitdist="mm" altunit="mm"/>
 <layers>
 <layer number="1" name="Top" color="4" fill="1" visible="yes" active="yes"/>
@@
 <hole x="2.5" y="37.5" drill="2"/>
 <hole x="37.5" y="37.5" drill="2"/>
-<text x="2.5" y="55" size="1.778" layer="25">FAME BOY DPAD</text>
-<text x="23.5" y="55" size="1.778" layer="26" rot="MR0">FAME BOY BAXY</text>
+<text x="9.5" y="56" size="1.778" layer="25">FAME BOY DPAD</text>
+<text x="30.5" y="56" size="1.778" layer="26" rot="MR0">FAME BOY BAXY</text>
 <text x="38.1" y="35.56" size="1.27" layer="25" rot="R180">The ugliest
 board
@@
 <element name="U$10" library="LOGOS" package="DAVEDARKO2_LOGO" value="" x="17.78" y="17.78"/>
 <element name="U$11" library="LOGOS" package="DAVEDARKO2_LOGO" value="" x="26.162" y="52.07"/>
+<element name="S2" library="SparkFun-Electromechanical" package="TACTILE-PTH-SIDE" value="SWITCH-MOMENTARY-2SIDE" x="6" y="57" rot="R180"/>
 </elements>
 <signals>
@@
 <wire x1="11.684" y1="25.146" x2="17.78" y2="25.146" width="0.1524" layer="16"/>
 <wire x1="17.78" y1="25.146" x2="19.30775625" y2="29.148575" width="0.1524" layer="16"/>
+<contactref element="S2" pad="1"/>
+<wire x1="8.5" y1="57" x2="9.9" y2="58.4" width="0.3048" layer="16"/>
+<wire x1="9.9" y1="58.4" x2="34.8" y2="58.4" width="0.3048" layer="16"/>
+<wire x1="34.8" y1="58.4" x2="36.2" y2="57" width="0.3048" layer="16"/>
+<wire x1="36.2" y1="57" x2="36.5" y2="57" width="0.3048" layer="16"/>
 </signal>
 <signal name="C4">
@@
 <wire x1="13.6525" y1="2.5" x2="13.6525" y2="4.1275" width="0.1524" layer="16"/>
 <wire x1="23.585040625" y1="44.16746875" x2="22.86" y2="45.72" width="0.1524" layer="1"/>
+<contactref element="S2" pad="2"/>
+<wire x1="3.5" y1="57" x2="8.636" y2="51.864" width="0.3048" layer="16"/>
+<wire x1="8.636" y1="51.864" x2="8.636" y2="49.53" width="0.3048" layer="16"/>
 </signal>
 <signal name="R4">
