File: Schematics/fameboy_button_pads.sch (EAGLE design)
At the start: 6 parts

Commit message: gerbers
Parts:
- S1: value SWITCH-MOMENTARY-2SIDE_EZ -> SWITCH-MOMENTARY-2SIDE; device SparkFun-Electromechanical:SWITCH-MOMENTARY-2SIDE_EZ -> SparkFun-Electromechanical:SWITCH-MOMENTARY-2SIDE
Changed lines of the file:
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@@
 <part name="U$3" library="parts" deviceset="SELECTSTART" device=""/>
 <part name="U$4" library="parts" deviceset="SELECTSTART" device=""/>
-<part name="S1" library="SparkFun-Electromechanical" deviceset="SWITCH-MOMENTARY-2" device="SIDE_EZ"/>
+<part name="S1" library="SparkFun-Electromechanical" deviceset="SWITCH-MOMENTARY-2" device="SIDE" value="SWITCH-MOMENTARY-2SIDE"/>
 <part name="JP1" library="SparkFun-Connectors" deviceset="M08" device=""/>
 </parts>

Commit message: double shoulder button
Parts:
- added S2: SWITCH-MOMENTARY-2SIDE, SparkFun-Electromechanical:SWITCH-MOMENTARY-2SIDE
Connections:
- net C3: now also S2.1
- net R3: now also S2.2
Changed lines of the file:
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@@
 <part name="S1" library="SparkFun-Electromechanical" deviceset="SWITCH-MOMENTARY-2" device="SIDE" value="SWITCH-MOMENTARY-2SIDE"/>
 <part name="JP1" library="SparkFun-Connectors" deviceset="M08" device=""/>
+<part name="S2" library="SparkFun-Electromechanical" deviceset="SWITCH-MOMENTARY-2" device="SIDE" value="SWITCH-MOMENTARY-2SIDE"/>
 </parts>
 <sheets>
@@
 <instance part="S1" gate="G$1" x="83.82" y="35.56"/>
 <instance part="JP1" gate="G$1" x="25.4" y="12.7" rot="R90"/>
+<instance part="S2" gate="G$1" x="83.82" y="40.64"/>
 </instances>
 <busses>
@@
 <segment>
 <pinref part="S1" gate="G$1" pin="1"/>
-<wire x1="78.74" y1="35.56" x2="55.88" y2="35.56" width="0.1524" layer="91"/>
+<wire x1="78.74" y1="35.56" x2="73.66" y2="35.56" width="0.1524" layer="91"/>
 <label x="55.88" y="35.56" size="1.016" layer="95" rot="R180" xref="yes"/>
+<pinref part="S2" gate="G$1" pin="1"/>
+<wire x1="73.66" y1="35.56" x2="55.88" y2="35.56" width="0.1524" layer="91"/>
+<wire x1="78.74" y1="40.64" x2="73.66" y2="40.64" width="0.1524" layer="91"/>
+<wire x1="73.66" y1="40.64" x2="73.66" y2="35.56" width="0.1524" layer="91"/>
+<junction x="73.66" y="35.56"/>
 </segment>
 <segment>
@@
 <pinref part="U$2" gate="G$1" pin="G_Y"/>
 <wire x1="35.56" y1="38.1" x2="33.02" y2="38.1" width="0.1524" layer="91"/>
-<wire x1="33.02" y1="38.1" x2="38.1" y2="38.1" width="0.1524" layer="91"/>
+<wire x1="33.02" y1="38.1" x2="35.56" y2="38.1" width="0.1524" layer="91"/>
 <label x="38.1" y="38.1" size="1.016" layer="95" xref="yes"/>
+<junction x="35.56" y="48.26"/>
+<junction x="35.56" y="43.18"/>
+<junction x="35.56" y="38.1"/>
+<wire x1="35.56" y1="38.1" x2="38.1" y2="38.1" width="0.1524" layer="91"/>
 </segment>
 <segment>
@@
 <wire x1="35.56" y1="66.04" x2="38.1" y2="66.04" width="0.1524" layer="91"/>
 <label x="38.1" y="66.04" size="1.016" layer="95" xref="yes"/>
+<junction x="35.56" y="71.12"/>
+<junction x="35.56" y="76.2"/>
+<junction x="35.56" y="66.04"/>
 </segment>
 <segment>
@@
 <pinref part="S1" gate="G$1" pin="2"/>
 <wire x1="88.9" y1="35.56" x2="101.6" y2="35.56" width="0.1524" layer="91"/>
-<wire x1="101.6" y1="35.56" x2="101.6" y2="50.8" width="0.1524" layer="91"/>
+<wire x1="101.6" y1="35.56" x2="101.6" y2="40.64" width="0.1524" layer="91"/>
 <label x="104.14" y="50.8" size="1.016" layer="95" xref="yes"/>
+<pinref part="S2" gate="G$1" pin="2"/>
+<wire x1="101.6" y1="40.64" x2="101.6" y2="50.8" width="0.1524" layer="91"/>
+<wire x1="88.9" y1="40.64" x2="101.6" y2="40.64" width="0.1524" layer="91"/>
+<junction x="101.6" y="68.58"/>
+<junction x="101.6" y="55.88"/>
+<junction x="101.6" y="50.8"/>
 </segment>
 <segment>
